File: hardware/HSDAC.kicad_pcb (KiCad board)
At the start: 2 copper layers, 70 x 24.6 mm, 75 parts, among them IC1 ES9018K2M, J1 SM07B-SRSS-TB__LF__SN_, J3 USB_C_Receptacle_USB2.0_16P, SW1 RST, U1 CH32V305FBP6, U2 ME6210A33M3G, U3 OPA1678, U4 OPA1678, U5 OPA1678, X1 8M

Commit message: fix exception when upload firmware
Parts:
- R7: value 470 -> 51
Changed lines of the file:
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@@
 			)
 		)
-		(property "Value" "470"
+		(property "Value" "51"
 			(at 0 1.43 0)
 			(layer "F.Fab")
